Commit message: new cypher_drone_description structure and corrected dims

File: isaac_ros-dev/src/cypher_drone_description/models/cypher/xacro/cameras.xacro (robot description, xacro)
@@ -1,18 +1,16 @@
-<?xml version="2.99"?>
-<robot xmlns:xacro="http://wiki.ros.org/xacro" name="cypher_cameras">
-  <xacro:property name="front_realsense_xyz"  value="0.09597 0.0475 0.1287"/>    <!-- mm -> m -->
-  <xacro:property name="left_realsense_xyz"   value="-0.0475 0.09597 0.09170"/>  <!-- mm -> m -->
-  <xacro:property name="right_realsense_xyz"  value="0.0475 -0.09597 0.09170"/>  <!-- mm -> m -->
-  <xacro:property name="front_cv_xyz"         value="0.05415 -0.03 0.08870"/>    <!-- mm -> m -->
-  <xacro:property name="down_cv_xyz"          value="0.03345 0 -0.027175"/>      <!-- mm -> m -->
-  <xacro:property name="rangefinder_xyz"      value="-0.001622 0.01792 -0.031257"/> <!-- mm -> m -->
-  <!-- Generic box camera macro -->
+<?xml version="3.0"?>
+<robot xmlns:xacro="http://wiki.ros.org/xacro" name="Cypher_Drone_V3">
+  <xacro:property name="front_realsense_xyz"  value="0.09597 0.0475 0.152542"/>
+  <xacro:property name="left_realsense_xyz"   value="-0.0475 0.09597 0.115542"/>
+  <xacro:property name="right_realsense_xyz"  value="0.0475 -0.09597 0.115542"/>
+  <xacro:property name="front_cv_xyz"         value="0.05415 -0.03 0.112524"/>
+  <xacro:property name="down_cv_xyz"          value="0.03345 0 -0.003333"/>
+  <xacro:property name="rangefinder_xyz"      value="-0.001622 0.01792 -0.10135"/>
   <xacro:macro name="simple_camera"
-               params="name parent xyz">
+               params="name parent xyz l_r l_p l_y j_r j_p j_y">
     <link name="${name}_link">
       <visual>
-        <origin xyz="0 0 0" rpy="0 0 0"/>
+        <origin xyz="0 0 0" rpy="${l_r} ${l_p} ${l_y}"/>
         <geometry>
-          <!-- Simple camera body representation -->
           <box size="0.04 0.02 0.02"/>
         </geometry>
@@ -22,5 +20,5 @@
       </visual>
       <collision>
-        <origin xyz="0 0 0" rpy="0 0 0"/>
+        <origin xyz="0 0 0" rpy="${l_r} ${l_p} ${l_y}"/>
         <geometry>
           <box size="0.04 0.02 0.02"/>
@@ -28,5 +26,5 @@
       </collision>
       <inertial>
-        <origin xyz="0 0 0" rpy="0 0 0"/>
+        <origin xyz="0 0 0" rpy="${l_r} ${l_p} ${l_y}"/>
         <mass value="0.05"/>
         <inertia
@@ -39,15 +37,13 @@
       <parent link="${parent}"/>
       <child  link="${name}_link"/>
-      <origin xyz="${xyz}" rpy="0 0 0"/>
+      <origin xyz="${xyz}" rpy="${j_r} ${j_p} ${j_y}"/>
     </joint>
   </xacro:macro>
-  <!-- Rangefinder macro (simple cylinder) -->
   <xacro:macro name="rangefinder"
-               params="name parent xyz">
+               params="name parent xyz j_r j_p j_y">
     <link name="${name}_link">
       <visual>
         <origin xyz="0 0 0" rpy="0 0 0"/>
         <geometry>
-          <!-- Stub representation of a small rangefinder -->
           <cylinder radius="0.01" length="0.03"/>
         </geometry>
@@ -74,40 +70,46 @@
       <parent link="${parent}"/>
       <child  link="${name}_link"/>
-      <origin xyz="${xyz}" rpy="0 0 0"/>
+      <origin xyz="${xyz}" rpy="${j_r} ${j_p} ${j_y}"/>
     </joint>
   </xacro:macro>
-  <!-- Convenience macro to spawn all vision sensors + rangefinder from base_link -->
   <xacro:macro name="cypher_cameras_block"
                params="parent">
-    <!-- Front RealSense (discrete) -->
     <xacro:simple_camera
       name="front_realsense"
       parent="${parent}"
-      xyz="${front_realsense_xyz}"/>
-    <!-- Left RealSense (discrete) -->
+      xyz="${front_realsense_xyz}"
+      l_r="0"  l_p="0"   l_y="0"
+      j_r="0"  j_p="0"   j_y="0"/>
     <xacro:simple_camera
       name="left_realsense"
       parent="${parent}"
-      xyz="${left_realsense_xyz}"/>
-    <!-- Right RealSense (discrete) -->
+      xyz="${left_realsense_xyz}"
+      l_r="0"      l_p="0"      l_y="0"
+      j_r="0"      j_p="0"      j_y="${pi/2}"/>
     <xacro:simple_camera
       name="right_realsense"
       parent="${parent}"
-      xyz="${right_realsense_xyz}"/>
-    <!-- Front CV camera -->
+      xyz="${right_realsense_xyz}"
+      l_r="0"       l_p="0"       l_y="0"
+      j_r="0"       j_p="0"       j_y="${-pi/2}"/>
     <xacro:simple_camera
       name="front_cv"
       parent="${parent}"
-      xyz="${front_cv_xyz}"/>
-    <!-- Downwards CV camera -->
+      xyz="${front_cv_xyz}"
+      l_r="${-pi/2}" l_p="0"       l_y="0"
+      j_r="${-pi/2}" j_p="0"       j_y="${-pi/2}"/>
     <xacro:simple_camera
       name="down_cv"
       parent="${parent}"
-      xyz="${down_cv_xyz}"/>
-    <!-- Rangefinder (new object) -->
+      xyz="${down_cv_xyz}"
+      l_r="0"        l_p="${pi}"   l_y="${pi/2}"
+      j_r="0"        j_p="${pi}"   j_y="${pi/2}"/>
     <xacro:rangefinder
       name="rangefinder"
       parent="${parent}"
-      xyz="${rangefinder_xyz}"/>
+      xyz="${rangefinder_xyz}"
+      j_r="0"
+      j_p="${pi/2}"
+      j_y="0"/>
   </xacro:macro>
 </robot>

File: isaac_ros-dev/src/cypher_drone_description/models/cypher/xacro/cypher.xacro (robot description, xacro)
@@ -1,13 +1,10 @@
-<?xml version="2.99"?>
-<robot xmlns:xacro="http://wiki.ros.org/xacro" name="cypher_drone_v2_99">
-  <!-- Include submodules -->
-  <xacro:include filename="$(find cypher_description)/urdf/propellers.xacro"/>
-  <xacro:include filename="$(find cypher_description)/urdf/cameras.xacro"/>
-  <!-- Basic body -->
+<?xml version="3.0"?>
+<robot xmlns:xacro="http://wiki.ros.org/xacro" name="Cypher_Drone_V3">
+  <xacro:include filename="$(find cypher_drone_description)/models/cypher/xacro/propellers.xacro"/>
+  <xacro:include filename="$(find cypher_drone_description)/models/cypher/xacro/cameras.xacro"/>
   <link name="base_link">
     <visual>
       <origin xyz="0 0 0" rpy="0 0 0"/>
       <geometry>
-        <!-- Simple body -->
         <box size="0.25 0.25 0.05"/>
       </geometry>
@@ -31,5 +28,4 @@
     </inertial>
   </link>
-  <!-- FMU/IMU frame -->
   <link name="imu_link"/>
   <joint name="base_link_to_imu" type="fixed">
@@ -38,10 +34,8 @@
     <origin xyz="0.042523 0.031 0.0735" rpy="0 0 0"/>
   </joint>
-  <!-- Propeller parameters -->
   <xacro:property name="prop_force_offset"          value="0.0"/>
   <xacro:property name="prop_housing_radius"        value="0.07"/>
   <xacro:property name="prop_housing_height"        value="0.02"/>
   <xacro:property name="prop_housing_center_offset" value="0.15"/>
-  <!-- Front-left propeller -->
   <xacro:propellers
       name="front_left"
@@ -53,5 +47,4 @@
       prop_housing_height="${prop_housing_height}"
       prop_housing_center_offset="${prop_housing_center_offset}"/>
-  <!-- Front-right propeller -->
   <xacro:propellers
       name="front_right"
@@ -63,5 +56,4 @@
       prop_housing_height="${prop_housing_height}"
       prop_housing_center_offset="${prop_housing_center_offset}"/>
-  <!-- Rear-left propeller -->
   <xacro:propellers
       name="rear_left"
@@ -73,5 +65,4 @@
       prop_housing_height="${prop_housing_height}"
       prop_housing_center_offset="${prop_housing_center_offset}"/>
-  <!-- Rear-right propeller -->
   <xacro:propellers
       name="rear_right"
@@ -83,5 +74,4 @@
       prop_housing_height="${prop_housing_height}"
       prop_housing_center_offset="${prop_housing_center_offset}"/>
-  <!-- Cameras + rangefinder block, all relative to base_link -->
   <xacro:cypher_cameras_block parent="base_link"/>
 </robot>

File: isaac_ros-dev/src/cypher_drone_description/models/cypher/xacro/propellers.xacro (robot description, xacro)
@@ -1,43 +1,46 @@
-<?xml version="1.0"?>
-<robot name="cypher_drone_v1-0" xmlns:xacro="http://wiki.ros.org/xacro">
-    <xacro:macro
-        name="propellers"
-        params="
-        name
-        parent
-        fb_reflect
-        lr_reflect
-        prop_force_offset
-        prop_housing_radius
-        prop_housing_height
-        prop_housing_center_offset
-        ">
-        <link name="${name}_propeller_link">
-            <visual>
-                <origin xyz="0 0 ${prop_force_offset}" rpy="0 0 0"/>
-                <geometry>
-                    <cylinder radius="${prop_housing_radius}" length="${prop_housing_height}" />
-                </geometry>
-                <material name="${name}_propeller-material" >
-                    <color rgba="0.107 0.003676 0.2747 1" />
-                </material>
-            </visual>
-            <collision>
-                <origin xyz="0 0 0.0091" rpy="0 0 0"/>
-                <geometry>
-                    <cylinder radius="${prop_housing_radius}" length="${prop_housing_height}" />
-                </geometry>
-            </collision>
-            <inertial>
-                <origin xyz="0 0 0.0091" rpy="0 0 0" />
-                <mass value="0.1" />
-                <inertia ixx="0.033333333" ixy="0" ixz="0" iyy="0.05" iyz="0" izz="0.033333333" />
-            </inertial>
-        </link>
-        <joint name="${parent}_to_${name}_propeller_link" type="fixed">
-            <parent link="${parent}"/>
-            <child link="${name}_propeller_link" />
-            <origin xyz="${fb_reflect * prop_housing_center_offset} ${lr_reflect * prop_housing_center_offset} 0" rpy="0 0 0" />
-        </joint>
-    </xacro:macro>
+<?xml version="3.0"?>
+<robot name="Cypher_Drone_V3" xmlns:xacro="http://wiki.ros.org/xacro">
+  <xacro:macro
+      name="propellers"
+      params="
+      name
+      parent
+      fb_reflect
+      lr_reflect
+      prop_force_offset
+      prop_housing_radius
+      prop_housing_height
+      prop_housing_center_offset
+      ">
+    <link name="${name}_propeller_link">
+      <visual>
+        <origin xyz="0 0 ${prop_force_offset}" rpy="0 0 0"/>
+        <geometry>
+          <cylinder radius="${prop_housing_radius}" length="${prop_housing_height}"/>
+        </geometry>
+        <material name="${name}_propeller-material">
+          <color rgba="0.107 0.003676 0.2747 1"/>
+        </material>
+      </visual>
+      <collision>
+        <origin xyz="0 0 0.0091" rpy="0 0 0"/>
+        <geometry>
+          <cylinder radius="${prop_housing_radius}" length="${prop_housing_height}"/>
+        </geometry>
+      </collision>
+      <inertial>
+        <origin xyz="0 0 0.0091" rpy="0 0 0"/>
+        <mass value="0.1"/>
+        <inertia
+          ixx="0.033333333" ixy="0" ixz="0"
+          iyy="0.05"       iyz="0"
+          izz="0.033333333"/>
+      </inertial>
+    </link>
+    <joint name="${parent}_to_${name}_propeller_link" type="fixed">
+      <parent link="${parent}"/>
+      <child  link="${name}_propeller_link"/>
+      <origin xyz="${fb_reflect * prop_housing_center_offset} ${lr_reflect * prop_housing_center_offset} 0" rpy="0 0 0"/>
+    </joint>
+  </xacro:macro>
 </robot>
