Commit message: description: remove top_visual_link and decommission cam_front pipeline
Front-facing CSI camera no longer exists on the airframe. Dropped the
top_visual_link + joint from arid.xacro, removed the cam_front pipeline
from gst_camera_manager's pipelines.yaml, and updated every doc/example
across the repo to the single-camera (cam_down) state.

File: local_ws/src/arid_description/urdf/arid.xacro (robot description, xacro)
@@ -57,10 +57,4 @@
   <xacro:realsense name="left"  x="-0.0175"  y="0.08875"  yaw="${pi/2}"/>
   <xacro:realsense name="right" x="0.0175"   y="-0.08875" yaw="${-pi/2}"/>
-  <link name="top_visual_link"/>
-  <joint name="base_link_to_top_visual_joint" type="fixed">
-    <parent link="base_link"/>
-    <child  link="top_visual_link"/>
-    <origin xyz="0.077 0.0 0.129792" rpy="${-pi/2} 0 ${-pi/2}"/>
-  </joint>
   <link name="bottom_visual_link"/>
   <joint name="base_link_to_bottom_visual_joint" type="fixed">
