Commit message: v1.3: full platform port — arid_supervisor, VSLAM hardening, cam_front resurrection, RSUSB-only librealsense, ROS_LOCALHOST_ONLY, new setup/scripts, ARID_v1.2 firmware
Forward-port of the complete upgraded ARID platform (SKID-lineage, landed via
v1.2_rslidar) adapted to the standard 3x RealSense + dual-IMX219 airframe:

- arid_supervisor: camera-proven VSLAM lifecycle (3-camera gate, one /reset_usb
  recovery, landed-gate on disable, /arid_supervisor/status, run_logs)
- VSLAM hardening: FSM-free reactor (reset-epoch -> reset_counter, stamp skew
  clamp, est_status lifecycle fix, launch-injected px4_vslam_reactor.yaml),
  vio_transform epoch forwarding, enable_sync:false + initial_reset:false x3
- cam_front resurrected (sensor-id 0, top_visual_link restored; cam_down back
  to sensor-id 1) + front/down selectors in verify, calibration, focus
- SKID 3-camera interactive config_realsense (front/left/right assignment)
- RSUSB-only librealsense policy (Dockerfile purge+pin, rosdep skip-keys,
  -Drealsense2_DIR pin, container self-heal); host uses pip pyrealsense2
- ROS_LOCALHOST_ONLY=1 everywhere + systemd DefaultEnvironment drop-in
- setup.sh rebuilt on the v1.2 base: menu/questionnaire/resume, pinned session
  logs + smoke logs, ZeroTier phase, user linger, nvpmodel hardening, uninstall
- new scripts: zt_join, colcon_isaac, colcon_local, in_isaac, wifi,
  update_submods, two-camera verify_cv_cams, cam_front-aware local_test
- foxglove-sdk submodule removed (apt foxglove bridge)
- usb_ros_reset.service <distro> boot bug fixed
- PX4: submodule -> a02da31b (4026_arid_quad_v1_2, UXRCE_DDS_PTCFG=1 default);
  prebuilt ARID_v1.2.px4 replaces ARID_v1.1.px4
- README rewritten; docs/archive.zip refreshed

Co-Authored-By: Claude Fable 5 <noreply@anthropic.com>

File: local_ws/src/arid_description/urdf/arid.xacro (robot description, xacro)
@@ -54,7 +54,15 @@
   <xacro:propeller name="rear_left"   x="${-propeller_span}" y="${propeller_span}"/>
   <xacro:propeller name="rear_right"  x="${-propeller_span}" y="${-propeller_span}"/>
+  <!-- Rotation-symmetric mount: left camera has NEGATIVE x / +y / yaw +pi/2, right camera
+       POSITIVE x / -y / yaw -pi/2. Magnitude (0.0175) is ARID-specific boom geometry. -->
   <xacro:realsense name="front" x="0.09875"  y="0.0175"   yaw="0"/>
   <xacro:realsense name="left"  x="-0.0175"  y="0.08875"  yaw="${pi/2}"/>
   <xacro:realsense name="right" x="0.0175"   y="-0.08875" yaw="${-pi/2}"/>
+  <link name="top_visual_link"/>
+  <joint name="base_link_to_top_visual_joint" type="fixed">
+    <parent link="base_link"/>
+    <child  link="top_visual_link"/>
+    <origin xyz="0.077 0.0 0.129792" rpy="${-pi/2} 0 ${-pi/2}"/>
+  </joint>
   <link name="bottom_visual_link"/>
   <joint name="base_link_to_bottom_visual_joint" type="fixed">
